Commit message: d405+gemini2 update

File: description/urdf/rebotarm_rs_with_d405.urdf.xacro (robot description, xacro)
@@ -14,12 +14,13 @@
       - D405 bottom: 1/4-20 at bottom_screw origin, two M3 at x=±10 mm (along hole line).
       - camera_xyz = hole midpoint; +X along hole pair, +Z along hole axis (into camera).
-      - mount_* = Gemini2 flange seed (same gripper interface).
+      - mount_* shared with Gemini2 (same gripper flange); align_mount syncs both.
+      - camera_* = D405-only (do not copy Gemini2 camera_*).
   -->
-  <xacro:property name="mount_xyz" value="-0.0857 0.0000 0.0002"/>
-  <xacro:property name="mount_rpy" value="1.5609 -0.0043 1.5333"/>
+  <xacro:property name="mount_xyz" value="-0.1201 0.0003 0.0507"/>
+  <xacro:property name="mount_rpy" value="1.5827 0.0024 1.5515"/>
   <xacro:property name="mount_mesh_scale" value="0.001 0.001 0.001"/>
-  <!-- Keep user-tuned orientation; snap position to mount hole midpoint (seated in red pocket). -->
-  <xacro:property name="camera_xyz" value="-0.0003 0.0463 -0.0081"/>
-  <xacro:property name="camera_rpy" value="-0.0444 -1.3136 -1.5225"/>
+  <!-- D405 seated in mount pocket (camera relative to camera_mount_link). -->
+  <xacro:property name="camera_xyz" value="-0.0003 0.0443 -0.0093"/>
+  <xacro:property name="camera_rpy" value="-0.0225 -1.0448 -1.5460"/>
   <link name="camera_mount_link">
     <visual>

File: description/urdf/rebotarm_rs_with_gemini2.urdf.xacro (robot description, xacro)
@@ -11,10 +11,10 @@
 # If you only use wrist_camera.launch.py (static TF), keep values in sync with
 # config/wrist_extrinsics.yaml.
-  <xacro:property name="mount_xyz" value="-0.0857 0.0000 0.0002"/>
-  <xacro:property name="mount_rpy" value="1.5609 -0.0043 1.5333"/>
+  <xacro:property name="mount_xyz" value="-0.1201 0.0003 0.0507"/>
+  <xacro:property name="mount_rpy" value="1.5827 0.0024 1.5515"/>
   <xacro:property name="mount_mesh_scale" value="0.001 0.001 0.001"/>
   <!-- Inverse of camera_botter_screw_joint: camera bottom screw at mount origin. -->
-  <xacro:property name="camera_xyz" value="0.0250 0.0542 0.0112"/>
-  <xacro:property name="camera_rpy" value="-0.0157 -1.3078 -1.5644"/>
+  <xacro:property name="camera_xyz" value="0.0249 0.0487 0.0090"/>
+  <xacro:property name="camera_rpy" value="0.0042 -1.0502 -1.5718"/>
   <link name="camera_mount_link">
     <visual>

Commit message: d405+gemini2 update urdf

File: description/urdf/rebotarm_rs_with_d405.urdf.xacro (robot description, xacro)
@@ -10,17 +10,12 @@
     Mount mesh: description/meshes/D405_305_Mount.stl (from D405_305_Mount.step, mm → scale 0.001).
     Frame chain: gripper_end -> camera_mount_link -> camera_bottom_screw_frame -> camera_link
-    Two-hole alignment (camera laid parallel into red pocket, not standing vertical):
-      - Mount face holes ~20 mm apart (STEP).
-      - D405 bottom: 1/4-20 at bottom_screw origin, two M3 at x=±10 mm (along hole line).
-      - camera_xyz = hole midpoint; +X along hole pair, +Z along hole axis (into camera).
-      - mount_* shared with Gemini2 (same gripper flange); align_mount syncs both.
-      - camera_* = D405-only (do not copy Gemini2 camera_*).
+    D405 uses its own mount CAD (not Gemini2's D435_Gemini2_Mount).
+    mount_* / camera_* are D405-only — do not sync from Gemini2.
   -->
-  <xacro:property name="mount_xyz" value="-0.1201 0.0003 0.0507"/>
-  <xacro:property name="mount_rpy" value="1.5827 0.0024 1.5515"/>
+  <xacro:property name="mount_xyz" value="-0.0857 0.0000 0.0002"/>
+  <xacro:property name="mount_rpy" value="1.5609 -0.0043 1.5333"/>
   <xacro:property name="mount_mesh_scale" value="0.001 0.001 0.001"/>
-  <!-- D405 seated in mount pocket (camera relative to camera_mount_link). -->
-  <xacro:property name="camera_xyz" value="-0.0003 0.0443 -0.0093"/>
-  <xacro:property name="camera_rpy" value="-0.0225 -1.0448 -1.5460"/>
+  <xacro:property name="camera_xyz" value="-0.0003 0.0463 -0.0081"/>
+  <xacro:property name="camera_rpy" value="-0.0444 -1.3136 -1.5225"/>
   <link name="camera_mount_link">
     <visual>

File: description/urdf/rebotarm_rs_with_gemini2.urdf.xacro (robot description, xacro)
@@ -11,5 +11,5 @@
 # If you only use wrist_camera.launch.py (static TF), keep values in sync with
 # config/wrist_extrinsics.yaml.
-  <xacro:property name="mount_xyz" value="-0.1201 0.0003 0.0507"/>
+  <xacro:property name="mount_xyz" value="-0.1201 0.0003 0.0450"/>
   <xacro:property name="mount_rpy" value="1.5827 0.0024 1.5515"/>
   <xacro:property name="mount_mesh_scale" value="0.001 0.001 0.001"/>

Commit message: D405 update

File: description/urdf/rebotarm_rs_with_d405.urdf.xacro (robot description, xacro)
@@ -13,9 +13,9 @@
     mount_* / camera_* are D405-only — do not sync from Gemini2.
   -->
-  <xacro:property name="mount_xyz" value="-0.0857 0.0000 0.0002"/>
-  <xacro:property name="mount_rpy" value="1.5609 -0.0043 1.5333"/>
+  <xacro:property name="mount_xyz" value="-0.1201 0.0003 0.0507"/>
+  <xacro:property name="mount_rpy" value="1.5827 0.0024 1.5515"/>
   <xacro:property name="mount_mesh_scale" value="0.001 0.001 0.001"/>
-  <xacro:property name="camera_xyz" value="-0.0003 0.0463 -0.0081"/>
-  <xacro:property name="camera_rpy" value="-0.0444 -1.3136 -1.5225"/>
+  <xacro:property name="camera_xyz" value="-0.0003 0.0443 -0.0093"/>
+  <xacro:property name="camera_rpy" value="-0.0225 -1.0448 -1.5460"/>
   <link name="camera_mount_link">
     <visual>
